File: Hardware/pcb_small/datalogger_pcb.kicad_sch (KiCad schematic)
At the start: 31 parts, among them J1 Micro_SD_Card_Det2, U1 DS3231MZ

Commit message: Small changes
Parts:
- removed Alim5V1: Bornier Alim, Connector_PinSocket_2.54mm:PinSocket_1x02_P2.54mm_Vertical, symbol Connector:Conn_01x02_Socket
- removed I2C0JST1: I2C 0 Connector, Connector_PinSocket_2.00mm:PinSocket_1x04_P2.00mm_Vertical, symbol Connector:Conn_01x04_Socket
- removed I2C1JST1: I2C 1 Connector, Connector_PinSocket_2.00mm:PinSocket_1x04_P2.00mm_Vertical, symbol Connector:Conn_01x04_Socket
- removed R5, R6: 10k, Resistor_SMD:R_0805_2012Metric_Pad1.20x1.40mm_HandSolder, symbol Device:R
- added I2C2: I2C 0 Connector, TerminalBlock_Phoenix:TerminalBlock_Phoenix_MKDS-1,5-4-5.08_1x04_P5.08mm_Horizontal, symbol Connector:Conn_01x04_Socket
- added RpullupCS1: 10k, Resistor_SMD:R_0805_2012Metric_Pad1.20x1.40mm_HandSolder, symbol Device:R
- added RpullupSCL1, RpullupSDA1: 10k, Resistor_THT:R_Axial_DIN0204_L3.6mm_D1.6mm_P5.08mm_Vertical, symbol Device:R
- added SW1: SW_Wuerth_450301014042, Button_Switch_THT:SW_Slide-03_Wuerth-WS-SLTV_10x2.5x6.4_P2.54mm, symbol Switch:SW_Wuerth_450301014042
- 5VPOUT1, PWR12V1: footprint Connector_PinSocket_2.54mm:PinSocket_1x02_P2.54mm_Vertical -> TerminalBlock_Phoenix:TerminalBlock_Phoenix_MKDS-1,5-2-5.08_1x02_P5.08mm_Horizontal
- GPIO10-1, GPIO14-1, GPIO6-1: footprint Connector_PinSocket_2.54mm:PinSocket_1x06_P2.54mm_Vertical -> TerminalBlock_Phoenix:TerminalBlock_Phoenix_MKDS-1,5-6-5.08_1x06_P5.08mm_Horizontal
- OneWire1: footprint Connector_PinSocket_2.54mm:PinSocket_1x03_P2.54mm_Vertical -> TerminalBlock_Phoenix:TerminalBlock_Phoenix_MKDS-1,5-3-5.08_1x03_P5.08mm_Horizontal
- UART1: footprint Connector_PinSocket_2.54mm:PinSocket_1x04_P2.54mm_Vertical -> TerminalBlock_Phoenix:TerminalBlock_Phoenix_MKDS-1,5-4-5.08_1x04_P5.08mm_Horizontal
Connections:
- net +12V: now also SW1.3 (A); no longer Alimoption1.4 (EN)
- net +3.3V: now also I2C2.4 (Pin_4), RpullupCS1.1, RpullupSCL1.1, RpullupSDA1.1; no longer GPIO6-1.6 (Pin_6)
- net CS: now also RpullupCS1.2
- net GND: now also I2C2.1 (Pin_1), SW1.2 (C); no longer GPIO6-1.1 (Pin_1)
- net I2C0_SCL: now also I2C2.3 (Pin_3)
- net I2C0_SDA: now also I2C2.2 (Pin_2)
- net I2C1_SCL: now also RpullupSCL1.2; no longer A1.5 (GPIO3)
- net I2C1_SDA: now also RpullupSDA1.2; no longer A1.4 (GPIO2)
- net at A1.20 (GPIO15), GPIO14-1.3 (Pin_3): no longer U1.3 (~{INT}/SQW)
- net at A1.27 (GPIO21), GPIO14-1.4 (Pin_4): no longer U1.1 (32KHZ)
- net at A1.11 (GPIO8): now also GPIO6-1.2 (Pin_2); no longer GPIO6-1.4 (Pin_4)
- net at A1.12 (GPIO9): now also GPIO6-1.1 (Pin_1); no longer GPIO6-1.5 (Pin_5)
- net at A1.9 (GPIO6): now also GPIO6-1.4 (Pin_4); no longer GPIO6-1.2 (Pin_2)
- new net: Alimoption1.4 (EN), SW1.1 (B)
- new net: A1.4 (GPIO2), GPIO6-1.6 (Pin_6)
- new net: A1.5 (GPIO3), GPIO6-1.5 (Pin_5)
Other:
- moved on the sheet: 5VPOUT1, C3, GPIO10-1, GPIO6-1, J1, OneWire1, Pullup_One_Wire1, R3, R4, UART1

Commit message: New smaller efficient pcb
Parts:
- removed 5VPOUT1: Bornier 5V, TerminalBlock_Phoenix:TerminalBlock_Phoenix_MKDS-1,5-2-5.08_1x02_P5.08mm_Horizontal, symbol Connector:Conn_01x02_Socket
- removed Alimoption1: ~, useful:TSOT-23-6_NEX, symbol useful:NEX_DC_DC
- removed BT1: Battery_Cell, Battery:BatteryHolder_Keystone_500, symbol Device:Battery_Cell
- removed C1: 100nF, Capacitor_SMD:C_1812_4532Metric_Pad1.57x3.40mm_HandSolder, symbol Device:C
- removed C2: 2.2µF, Capacitor_SMD:C_1812_4532Metric_Pad1.57x3.40mm_HandSolder, symbol Device:C
- removed C3: 22µF, Capacitor_SMD:C_1812_4532Metric_Pad1.57x3.40mm_HandSolder, symbol Device:C
- removed GPIO10-1: GPIO10-13, TerminalBlock_Phoenix:TerminalBlock_Phoenix_MKDS-1,5-6-5.08_1x06_P5.08mm_Horizontal, symbol Connector:Conn_01x06_Socket
- removed GPIO14-1: GPIO14-17, TerminalBlock_Phoenix:TerminalBlock_Phoenix_MKDS-1,5-6-5.08_1x06_P5.08mm_Horizontal, symbol Connector:Conn_01x06_Socket
- removed GPIO6-1: GPIO6-9, TerminalBlock_Phoenix:TerminalBlock_Phoenix_MKDS-1,5-6-5.08_1x06_P5.08mm_Horizontal, symbol Connector:Conn_01x06_Socket
- removed I2C2: I2C 0 Connector, TerminalBlock_Phoenix:TerminalBlock_Phoenix_MKDS-1,5-4-5.08_1x04_P5.08mm_Horizontal, symbol Connector:Conn_01x04_Socket
- removed L_alim1: 18µH, Inductor_SMD:L_TracoPower_TCK-047_5.2x5.8mm, symbol Device:L
- removed OneWire1: Connecteur OneWire, TerminalBlock_Phoenix:TerminalBlock_Phoenix_MKDS-1,5-3-5.08_1x03_P5.08mm_Horizontal, symbol Connector:Conn_01x03_Socket
- removed PWR12V1: 12V PWR, TerminalBlock_Phoenix:TerminalBlock_Phoenix_MKDS-1,5-2-5.08_1x02_P5.08mm_Horizontal, symbol Connector:Conn_01x02_Socket
- removed R3: 105k, Resistor_SMD:R_0805_2012Metric_Pad1.20x1.40mm_HandSolder, symbol Device:R
- removed R4: 20k, Resistor_SMD:R_0805_2012Metric_Pad1.20x1.40mm_HandSolder, symbol Device:R
- removed SW1: SW_Wuerth_450301014042, Button_Switch_THT:SW_Slide-03_Wuerth-WS-SLTV_10x2.5x6.4_P2.54mm, symbol Switch:SW_Wuerth_450301014042
- removed UART1: UART Connector, TerminalBlock_Phoenix:TerminalBlock_Phoenix_MKDS-1,5-4-5.08_1x04_P5.08mm_Horizontal, symbol Connector:Conn_01x04_Socket
- added I2C0JST1: I2C 0 Connector, Connector_PinSocket_2.00mm:PinSocket_1x04_P2.00mm_Vertical, symbol Connector:Conn_01x04_Socket
- added J5: Conn_01x10_Socket, TerminalBlock_Phoenix:TerminalBlock_Phoenix_MKDS-1-10-3.81_1x10_P3.81mm_Horizontal, symbol Connector:Conn_01x10_Socket
- added P_MOSFET1, Q1: Si2319CDS, Package_TO_SOT_SMD:SOT-23, symbol Transistor_FET:Si2319CDS
- added R8, R_pullup_int1, R_pullup_shtdwn1: 100k, Resistor_SMD:R_0805_2012Metric_Pad1.20x1.40mm_HandSolder, symbol Device:R
- added R_BYPASS1: 0 Ohm, Resistor_SMD:R_0805_2012Metric_Pad1.20x1.40mm_HandSolder, symbol Device:R
- added SW2: SW_Push, Button_Switch_THT:SW_PUSH_6mm_H4.3mm, symbol Switch:SW_Push
- added U2: SN74LVC2G00DCTR, nand:SSOP-8_2.95x2.8mm_P0.65mm - SN74LVC2G00, symbol SN74LVC2G00DCTR:SN74LVC2G00DCTR
Connections:
- net Batt+ is gone; now on net BATT: U1.6 (VBAT)
- net +3.3V: now also I2C0JST1.3 (Pin_3), J5.10 (Pin_10)
- net Data_Onewire: now also A1.9 (GPIO6), J5.3 (Pin_3); no longer A1.29 (GPIO22)
- net GND: now also I2C0JST1.4 (Pin_4), J5.1 (Pin_1), R8.2, SW2.1, U2.4 (GND)
- net I2C0_SCL: now also I2C0JST1.1 (Pin_1), J5.9 (Pin_9)
- net I2C0_SDA: now also I2C0JST1.2 (Pin_2), J5.8 (Pin_8)
- net I2C1_SCL: now also A1.5 (GPIO3), J5.7 (Pin_7)
- net I2C1_SDA: now also A1.4 (GPIO2), J5.6 (Pin_6)
- net UART0_RX: now also J5.5 (Pin_5)
- net UART0_TX: now also J5.4 (Pin_4)
- net at F1.2: now also Q1.2 (S); no longer PWRIN1.2 (Pin_2)
- net SHTDWN_CTRL: now reaches A1.27 (GPIO21)
- net SHTDWN_CTRL: now also R_pullup_int1.2, U2.1 (1A)
- net RTC_INT: now reaches U1.3 (~{INT}/SQW)
- net RTC_INT: now also R_pullup_shtdwn1.1, SW2.2, U2.5 (2A)
- net +12V renamed BATT
- net BATT: now also P_MOSFET1.3 (D), R_BYPASS1.1, R_pullup_int1.1, R_pullup_shtdwn1.2, U2.8 (VCC); no longer R1.1
- net +5V renamed +5VP
- net +5VP: now also P_MOSFET1.2 (S), R_BYPASS1.2
- new net: P_MOSFET1.1 (G), U2.6 (2B), U2.7 (1Y)
- new net: Q1.1 (G), R8.1
- new net: U2.2 (1B), U2.3 (2Y)
- new net BATTREAD: PWRIN1.2 (Pin_2), Q1.3 (D), R1.1
Other:
- moved on the sheet: C4, F1, J1, Pullup_One_Wire1, Rpllup1, Rpllup2, RpullupCS1, RpullupSCL1, RpullupSDA1, U1

Commit message: Changes in small pcb
Parts:
- added C1: 100nF, Capacitor_SMD:C_1812_4532Metric_Pad1.57x3.40mm_HandSolder, symbol Device:C
- added C2: 10µF, Capacitor_SMD:C_1812_4532Metric_Pad1.57x3.40mm_HandSolder, symbol Device:C
- added C5: 100uF, Capacitor_SMD:C_1812_4532Metric_Pad1.57x3.40mm_HandSolder, symbol Device:C
- added D1: SS14, Diode_SMD:D_SMA, symbol Diode:SS14
- PWRIN1: value 7-48V Alim -> Batteries
- R1: value 68k -> 100k
- R2: value 22k -> 10k
- R_pullup_int1: value 100k -> 1M
Connections:
- net +3.3V: now also C2.1
- net BATT: now also P_MOSFET1.2 (S), C1.1; no longer P_MOSFET1.3 (D)
- net GND: now also C1.2, C2.2, C5.2
- net SHTDWN_CTRL: now also R1.2; no longer A1.27 (GPIO21)
- net at U2.6 (2B), U2.7 (1Y): now also R2.2; no longer P_MOSFET1.1 (G)
- net +5VP: no longer names the net of A1.39 (VSYS), R_BYPASS1.2
- net +5VP: now also C5.1, D1.1 (K); no longer P_MOSFET1.2 (S)
- net AGND: no longer names the net of A1.33 (AGND)
- net AGND: no longer R2.2
- net BATTREAD: no longer names the net of PWRIN1.2 (Pin_2), Q1.3 (D)
- net BATTREAD: no longer R1.1
- removed net READ12V: A1.31 (GPIO26_ADC0), R1.2, R2.1
- new net: A1.27 (GPIO21), R1.1
- new net: P_MOSFET1.1 (G), R2.1
- new net: D1.2 (A), P_MOSFET1.3 (D)
Other:
- moved on the sheet: F1, PWRIN1, P_MOSFET1, Q1, R8, R_BYPASS1

Commit message: Changes to ulogger pcb
Parts:
- added BT1: Battery_Cell, Battery:BatteryHolder_Keystone_500, symbol Device:Battery_Cell
- added Q2: 2N7002, Package_TO_SOT_SMD:SOT-23, symbol Transistor_FET:2N7002
- added R3: 100k, Resistor_SMD:R_0805_2012Metric_Pad1.20x1.40mm_HandSolder, symbol Device:R
- R1: value 100k -> 10k
Connections:
- net BATT: no longer U1.6 (VBAT)
- net GND: now also BT1.2 (-), R3.2
- net SHTDWN_CTRL: now also Q2.3 (D); no longer R1.2
- net at A1.20 (GPIO15): now also J5.2 (Pin_2)
- net at A1.27 (GPIO21): no longer R1.1
- net at A1.29 (GPIO22): now also R1.1
- new net: BT1.1 (+), U1.6 (VBAT)
- new net: Q2.1 (G), R1.2
- new net: Q2.2 (S), R3.1
Other:
- moved on the sheet: C2, Pullup_One_Wire1, R1, RpullupCS1

Commit message: Changes to small pcb
Parts:
- removed R_BYPASS1: 0 Ohm, Resistor_SMD:R_0805_2012Metric_Pad1.20x1.40mm_HandSolder, symbol Device:R
- added C3: 100 µF, Capacitor_THT:CP_Radial_D7.5mm_P2.50mm, symbol Device:C_Polarized
- C1, C4: footprint Capacitor_SMD:C_1812_4532Metric_Pad1.57x3.40mm_HandSolder -> Capacitor_SMD:C_1206_3216Metric_Pad1.33x1.80mm_HandSolder
- C5: value 100uF -> 10 µF
Connections:
- net BATT: now also C5.1
- net GND: now also Q2.2 (S), C3.2
- net at A1.39 (VSYS), D1.1 (K): now also C3.1; no longer C5.1
- net at Q2.1 (G), R1.2: now also R3.1
Other:
- moved on the sheet: R3
