File: Hardware/pcb_small/datalogger_pcb.kicad_pcb (KiCad board)
At the start: 2 copper layers, 72.5 x 61.9 mm, 31 parts, among them J1 Micro_SD_Card_Det2, U1 DS3231MZ

Commit message: Small changes
Parts:
- removed 12VOUT: 12V PWR, Connector_PinSocket_2.54mm:PinSocket_1x02_P2.54mm_Vertical
- removed 5VIN: Bornier Alim, Connector_PinSocket_2.54mm:PinSocket_1x02_P2.54mm_Vertical
- removed 5VOUT: Bornier 5V, Connector_PinSocket_2.54mm:PinSocket_1x02_P2.54mm_Vertical
- removed GPIO 6-9: GPIO6-9, Connector_PinSocket_2.54mm:PinSocket_1x06_P2.54mm_Vertical
- removed GPIO10-13: GPIO10-13, Connector_PinSocket_2.54mm:PinSocket_1x06_P2.54mm_Vertical
- removed GPIO14-15-21-27: GPIO14-17, Connector_PinSocket_2.54mm:PinSocket_1x06_P2.54mm_Vertical
- removed I2C0JST1: I2C 0 Connector, Connector_PinSocket_2.00mm:PinSocket_1x04_P2.00mm_Vertical
- removed I2C1JST1: I2C 1 Connector, Connector_PinSocket_2.00mm:PinSocket_1x04_P2.00mm_Vertical
- removed R5, R6: 10k, Resistor_SMD:R_0805_2012Metric_Pad1.20x1.40mm_HandSolder
- added 5VPOUT1: Bornier 5V, TerminalBlock_Phoenix:TerminalBlock_Phoenix_MKDS-1,5-2-5.08_1x02_P5.08mm_Horizontal, B.Cu at (148.8, 38.4)
- added GPIO10-1: GPIO10-13, TerminalBlock_Phoenix:TerminalBlock_Phoenix_MKDS-1,5-6-5.08_1x06_P5.08mm_Horizontal, B.Cu at (146.7, 70.5)
- added GPIO14-1: GPIO14-17, TerminalBlock_Phoenix:TerminalBlock_Phoenix_MKDS-1,5-6-5.08_1x06_P5.08mm_Horizontal, B.Cu at (301.4, 44.4)
- added GPIO6-1: GPIO6-9, TerminalBlock_Phoenix:TerminalBlock_Phoenix_MKDS-1,5-6-5.08_1x06_P5.08mm_Horizontal, B.Cu at (132.7, 96.2)
- added I2C2: I2C 0 Connector, TerminalBlock_Phoenix:TerminalBlock_Phoenix_MKDS-1,5-4-5.08_1x04_P5.08mm_Horizontal, B.Cu at (146.9, 48.6)
- added PWR12V1: 12V PWR, TerminalBlock_Phoenix:TerminalBlock_Phoenix_MKDS-1,5-2-5.08_1x02_P5.08mm_Horizontal, B.Cu at (136.1, 38.4)
- added RpullupCS1: 10k, Resistor_SMD:R_0805_2012Metric_Pad1.20x1.40mm_HandSolder, F.Cu at (118.5, 77.0)
- added RpullupSCL1: 10k, Resistor_THT:R_Axial_DIN0204_L3.6mm_D1.6mm_P5.08mm_Vertical, F.Cu at (105.7, 100.1)
- added RpullupSDA1: 10k, Resistor_THT:R_Axial_DIN0204_L3.6mm_D1.6mm_P5.08mm_Vertical, F.Cu at (105.7, 103.3)
- added SW1: SW_Wuerth_450301014042, Button_Switch_THT:SW_Slide-03_Wuerth-WS-SLTV_10x2.5x6.4_P2.54mm, F.Cu at (116.9, 40.4)
- A1, PWRIN1: moved to B.Cu
- OneWire1: footprint Connector_PinSocket_2.54mm:PinSocket_1x03_P2.54mm_Vertical -> TerminalBlock_Phoenix:TerminalBlock_Phoenix_MKDS-1,5-3-5.08_1x03_P5.08mm_Horizontal; moved to B.Cu
- UART1: footprint Connector_PinSocket_2.54mm:PinSocket_1x04_P2.54mm_Vertical -> TerminalBlock_Phoenix:TerminalBlock_Phoenix_MKDS-1,5-4-5.08_1x04_P5.08mm_Horizontal; moved to B.Cu
- moved UART1 85.3 mm to (133.5, 48.5), turned to -90 degrees
- moved A1 68.9 mm to (124.5, 45.2), turned to 180 degrees
- moved C2 53.6 mm to (119.2, 47.8), turned to 180 degrees
- moved BT1 52.7 mm to (96.2, 92.5), turned to 90 degrees
- moved F1 52.6 mm to (125.8, 41.9), turned to 90 degrees
- moved R4 49.5 mm to (121.2, 61.4), turned to -90 degrees
- moved C1 48.6 mm to (114.8, 61.7), turned to 0 degrees
- moved Alimoption1 48.1 mm to (120.3, 53.9)
- moved R3 43.8 mm to (120.2, 58.0), turned to 0 degrees
- moved R1 40.1 mm to (112.4, 61.7), turned to 180 degrees
- moved R2 38.7 mm to (112.4, 59.6)
- moved OneWire1 37.9 mm to (97.1, 50.3)
- moved Rpllup1 33.7 mm to (119.5, 67.3)
- moved C3 33.5 mm to (112.2, 47.8)
- moved L_alim1 33.3 mm to (113.4, 53.8), turned to 90 degrees
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Connections:
- A1 pad 4: /I2C1_SDA -> Net-(A1-GPIO2)
- A1 pad 5: /I2C1_SCL -> Net-(A1-GPIO3)
- Alimoption1 pad 4: +12V -> Net-(Alimoption1-EN)
- U1 pad 1: Net-(A1-GPIO21) -> unconnected-(U1-32KHZ-Pad1)
- U1 pad 3: Net-(A1-GPIO15) -> unconnected-(U1-~{INT}/SQW-Pad3)
Routing:
- net +3.3V: track 212.1 -> 110.2 mm, vias 0 -> 3
- net /Data_Onewire: track 99.3 -> 20.8 mm
- net Net-(A1-GPIO27_ADC1): track 73.1 -> 0.00 mm
- net Net-(A1-GPIO21): track 53.7 -> 0.00 mm, vias 1 -> 0
- net GND: track 0.00 -> 46.1 mm, vias 16 -> 0
- net Net-(A1-GPIO11): track 31.8 -> 0.00 mm
- net Net-(A1-GPIO15): track 30.3 -> 0.00 mm, vias 1 -> 0
- net Net-(A1-GPIO10): track 30.2 -> 0.00 mm
- net +12V: track 70.2 -> 44.1 mm, vias 0 -> 2
- net Net-(A1-GPIO12): track 20.2 -> 0.00 mm
- net Net-(A1-GPIO13): track 19.7 -> 0.00 mm
- net /SCK: track 32.8 -> 13.5 mm, vias 1 -> 0
- net Net-(PWRIN1-Pin_2): track 6.51 -> 25.3 mm
- net /Batt+: track 36.2 -> 55.0 mm, vias 2 -> 3
- net /CS: track 16.7 -> 30.5 mm, vias 0 -> 2
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- removed copper zone on B.Cu, net GND
- removed copper zone on F.Cu, net GND
Other:
- board outline removed
- board text removed: "+"
- board text removed: "-"
- board text removed: "100nF"
- board text removed: "105k"
- board text removed: "10k"
- board text removed: "18µH"
- board text removed: "2.2µF"
- board text removed: "20k"
- board text removed: "22k"
- board text removed: "22µF"
- board text removed: "3.3"
- board text removed: "68k"
- board text removed: "BATT PWR"
- board text removed: "CL"
- board text removed: "DA"
- board text removed: "DS3231MZ"
- board text removed: "G"
- board text removed: "I2C0 JST"
- board text removed: "I2C1 JST"
- board text removed: "M2"
- board text removed: "NEX40400ADAZ"
- board text removed: "RX"
- board text removed: "SD Card"
- board text removed: "TX"
- board text removed: "µDlggr"

Commit message: New smaller efficient pcb
Parts:
- removed 5VPOUT1: Bornier 5V, TerminalBlock_Phoenix:TerminalBlock_Phoenix_MKDS-1,5-2-5.08_1x02_P5.08mm_Horizontal
- removed Alimoption1: ~, useful:TSOT-23-6_NEX
- removed BT1: Battery_Cell, Battery:BatteryHolder_Keystone_500
- removed C1: 100nF, Capacitor_SMD:C_1812_4532Metric_Pad1.57x3.40mm_HandSolder
- removed C2: 2.2µF, Capacitor_SMD:C_1812_4532Metric_Pad1.57x3.40mm_HandSolder
- removed C3: 22µF, Capacitor_SMD:C_1812_4532Metric_Pad1.57x3.40mm_HandSolder
- removed GPIO10-1: GPIO10-13, TerminalBlock_Phoenix:TerminalBlock_Phoenix_MKDS-1,5-6-5.08_1x06_P5.08mm_Horizontal
- removed GPIO14-1: GPIO14-17, TerminalBlock_Phoenix:TerminalBlock_Phoenix_MKDS-1,5-6-5.08_1x06_P5.08mm_Horizontal
- removed GPIO6-1: GPIO6-9, TerminalBlock_Phoenix:TerminalBlock_Phoenix_MKDS-1,5-6-5.08_1x06_P5.08mm_Horizontal
- removed I2C2: I2C 0 Connector, TerminalBlock_Phoenix:TerminalBlock_Phoenix_MKDS-1,5-4-5.08_1x04_P5.08mm_Horizontal
- removed L_alim1: 18µH, Inductor_SMD:L_TracoPower_TCK-047_5.2x5.8mm
- removed OneWire1: Connecteur OneWire, TerminalBlock_Phoenix:TerminalBlock_Phoenix_MKDS-1,5-3-5.08_1x03_P5.08mm_Horizontal
- removed PWR12V1: 12V PWR, TerminalBlock_Phoenix:TerminalBlock_Phoenix_MKDS-1,5-2-5.08_1x02_P5.08mm_Horizontal
- removed R3: 105k, Resistor_SMD:R_0805_2012Metric_Pad1.20x1.40mm_HandSolder
- removed R4: 20k, Resistor_SMD:R_0805_2012Metric_Pad1.20x1.40mm_HandSolder
- removed SW1: SW_Wuerth_450301014042, Button_Switch_THT:SW_Slide-03_Wuerth-WS-SLTV_10x2.5x6.4_P2.54mm
- removed UART1: UART Connector, TerminalBlock_Phoenix:TerminalBlock_Phoenix_MKDS-1,5-4-5.08_1x04_P5.08mm_Horizontal
- added I2C0JST1: I2C 0 Connector, Connector_PinSocket_2.00mm:PinSocket_1x04_P2.00mm_Vertical, F.Cu at (93.5, 82.0)
- added J5: Conn_01x10_Socket, TerminalBlock_Phoenix:TerminalBlock_Phoenix_MKDS-1-10-3.81_1x10_P3.81mm_Horizontal, F.Cu at (86.3, 48.0)
- added P_MOSFET1: Si2319CDS, Package_TO_SOT_SMD:SOT-23, F.Cu at (128.0, 76.9)
- added Q1: Si2319CDS, Package_TO_SOT_SMD:SOT-23, F.Cu at (129.0, 58.5)
- added R8: 100k, Resistor_SMD:R_0805_2012Metric_Pad1.20x1.40mm_HandSolder, F.Cu at (125.0, 59.4)
- added R_BYPASS1: 0 Ohm, Resistor_SMD:R_0805_2012Metric_Pad1.20x1.40mm_HandSolder, F.Cu at (125.2, 67.0)
- added R_pullup_int1: 100k, Resistor_SMD:R_0805_2012Metric_Pad1.20x1.40mm_HandSolder, F.Cu at (121.5, 79.1)
- added R_pullup_shtdwn1: 100k, Resistor_SMD:R_0805_2012Metric_Pad1.20x1.40mm_HandSolder, F.Cu at (126.9, 83.9)
- added SW2: SW_Push, Button_Switch_THT:SW_PUSH_6mm_H4.3mm, F.Cu at (129.8, 91.1)
- added U2: SN74LVC2G00DCTR, nand:SSOP-8_2.95x2.8mm_P0.65mm - SN74LVC2G00, F.Cu at (126.0, 81.1)
- A1, PWRIN1: moved to F.Cu
- moved RpullupSDA1 40.6 mm to (92.5, 64.9), turned to 90 degrees
- moved RpullupSCL1 37.7 mm to (96.9, 63.5), turned to 90 degrees
- moved PWRIN1 32.0 mm to (124.0, 51.2)
- moved F1 25.5 mm to (129.1, 67.2)
- moved A1 25.0 mm to (99.6, 47.1), turned to 0 degrees
- moved Rpllup1 17.2 mm to (103.3, 61.3), turned to 180 degrees
- moved RpullupCS1 17.0 mm to (120.9, 93.8), turned to 90 degrees
- moved R1 13.0 mm to (121.5, 71.0), turned to 90 degrees
- moved Rpllup2 12.3 mm to (105.0, 71.0), turned to 90 degrees
- moved R2 11.0 mm to (121.5, 65.9), turned to 90 degrees
- moved Pullup_One_Wire1 9.32 mm to (96.7, 72.7), turned to 90 degrees
- moved J1 8.75 mm to (108.5, 92.3)
- moved U1 7.14 mm to (107.6, 66.2), turned to 180 degrees
- moved C4 3.22 mm to (110.4, 71.2), turned to 0 degrees
Connections:
- A1 pad 10: Net-(A1-GPIO7) -> unconnected-(A1-GPIO7-Pad10)
- A1 pad 11: Net-(A1-GPIO8) -> unconnected-(A1-GPIO8-Pad11)
- A1 pad 12: Net-(A1-GPIO9) -> unconnected-(A1-GPIO9-Pad12)
- A1 pad 14: Net-(A1-GPIO10) -> unconnected-(A1-GPIO10-Pad14)
- A1 pad 15: Net-(A1-GPIO11) -> unconnected-(A1-GPIO11-Pad15)
- A1 pad 16: Net-(A1-GPIO12) -> unconnected-(A1-GPIO12-Pad16)
- A1 pad 17: Net-(A1-GPIO13) -> unconnected-(A1-GPIO13-Pad17)
- A1 pad 19: Net-(A1-GPIO14) -> unconnected-(A1-GPIO14-Pad19)
- A1 pad 20: Net-(A1-GPIO15) -> unconnected-(A1-GPIO15-Pad20)
- A1 pad 27: Net-(A1-GPIO21) -> /SHTDWN_CTRL
- A1 pad 29: /Data_Onewire -> unconnected-(A1-GPIO22-Pad29)
- A1 pad 32: Net-(A1-GPIO27_ADC1) -> unconnected-(A1-GPIO27_ADC1-Pad32)
- A1 pad 39: +5V -> +5VP
- A1 pad 4: Net-(A1-GPIO2) -> /I2C1_SDA
- A1 pad 5: Net-(A1-GPIO3) -> /I2C1_SCL
- A1 pad 9: Net-(A1-GPIO6) -> /Data_Onewire
- F1 pad 1: +12V -> /BATT
- F1 pad 2: Net-(PWRIN1-Pin_2) -> Net-(Q1-S)
- PWRIN1 pad 2: Net-(PWRIN1-Pin_2) -> /BATTREAD
- R1 pad 1: +12V -> /BATTREAD
- U1 pad 3: unconnected-(U1-~{INT}/SQW-Pad3) -> /RTC_INT
- U1 pad 6: /Batt+ -> /BATT
Routing:
- net /BATT: track 0.00 -> 89.5 mm, vias 0 -> 2
- net /RTC_INT: track 0.00 -> 80.4 mm, vias 0 -> 1
- net +5V: track 76.0 -> 0.00 mm, vias 2 -> 0
- net /Data_Onewire: track 20.8 -> 86.8 mm
- net /I2C0_SCL: track 35.9 -> 96.9 mm, vias 1 -> 3
- net /Batt+: track 55.0 -> 0.00 mm, vias 3 -> 0
- net GND: track 46.1 -> 0.00 mm, vias 0 -> 4
- net +12V: track 44.1 -> 0.00 mm, vias 2 -> 0
- net /I2C0_SDA: track 44.8 -> 86.8 mm, vias 1 -> 0
- net +3.3V: track 110.2 -> 149.8 mm, vias 3 -> 2
- net /BATTREAD: track 0.00 -> 38.6 mm
- net +5VP: track 0.00 -> 31.0 mm, vias 0 -> 2
- net /I2C1_SCL: track 0.00 -> 25.7 mm
- net Net-(PWRIN1-Pin_2): track 25.3 -> 0.00 mm
- net /I2C1_SDA: track 0.00 -> 19.6 mm
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- added copper zone on B.Cu, net GND
- added copper zone on F.Cu, net GND
Other:
- board outline added: 55 x 67 mm

Commit message: Changes in small pcb
Parts:
- added C1: 100nF, Capacitor_SMD:C_1812_4532Metric_Pad1.57x3.40mm_HandSolder, F.Cu at (128.2, 71.3)
- added C2: 10µF, Capacitor_SMD:C_1812_4532Metric_Pad1.57x3.40mm_HandSolder, F.Cu at (110.6, 80.8)
- added C5: 100uF, Capacitor_SMD:C_1812_4532Metric_Pad1.57x3.40mm_HandSolder, F.Cu at (123.0, 63.0)
- added D1: SS14, Diode_SMD:D_SMA, F.Cu at (122.4, 69.4)
- PWRIN1: value 7-48V Alim -> Batteries
- R1: value 68k -> 100k
- R2: value 22k -> 10k
- R_pullup_int1: value 100k -> 1M
- moved R2 17.5 mm to (131.3, 80.4), turned to -90 degrees
- moved R1 9.25 mm to (121.5, 80.2), turned to 0 degrees
- moved R_pullup_int1 6.17 mm to (124.1, 84.7), turned to 180 degrees
- moved P_MOSFET1 5.05 mm to (123.2, 75.1), turned to 180 degrees
- moved SW2 1.54 mm to (130.7, 92.3)
- moved F1 1.53 mm to (130.6, 67.4)
- moved R_pullup_shtdwn1 1.44 mm to (128.0, 84.8)
- moved R8 1.37 mm to (126.1, 58.5), turned to 90 degrees
- moved R_BYPASS1 1.08 mm to (126.2, 67.4)
- moved U2 0.40 mm to (126.4, 81.2)
Connections:
- A1 pad 27: /SHTDWN_CTRL -> Net-(A1-GPIO21)
- A1 pad 31: /READ12V -> unconnected-(A1-GPIO26_ADC0-Pad31)
- A1 pad 33: /AGND -> unconnected-(A1-AGND-Pad33)
- A1 pad 39: +5VP -> Net-(A1-VSYS)
- PWRIN1 pad 2: /BATTREAD -> Net-(PWRIN1-Pin_2)
- P_MOSFET1 pad 2: +5VP -> /BATT
- P_MOSFET1 pad 3: /BATT -> Net-(D1-A)
- Q1 pad 3: /BATTREAD -> Net-(PWRIN1-Pin_2)
- R1 pad 1: /BATTREAD -> Net-(A1-GPIO21)
- R1 pad 2: /READ12V -> /SHTDWN_CTRL
- R2 pad 1: /READ12V -> Net-(P_MOSFET1-G)
- R2 pad 2: /AGND -> Net-(U2-1Y)
- R_BYPASS1 pad 2: +5VP -> Net-(A1-VSYS)
- U2 pad 6: Net-(P_MOSFET1-G) -> Net-(U2-1Y)
- U2 pad 7: Net-(P_MOSFET1-G) -> Net-(U2-1Y)
Routing:
- net /BATTREAD: track 38.6 -> 0.00 mm
- net +5VP: track 31.0 -> 0.00 mm, vias 2 -> 0
- net Net-(A1-VSYS): track 0.00 -> 25.8 mm
- net Net-(PWRIN1-Pin_2): track 0.00 -> 7.69 mm
- net /READ12V: track 7.22 -> 0.00 mm
- net /AGND: track 4.11 -> 0.00 mm
- net Net-(U2-1Y): track 0.00 -> 3.95 mm
- net Net-(D1-A): track 0.00 -> 3.72 mm
- net Net-(A1-GPIO21): track 0.00 -> 3.27 mm
- net /RTC_INT: track 80.4 -> 83.2 mm
- net Net-(P_MOSFET1-G): track 11.8 -> 9.76 mm
- net /BATT: track 89.5 -> 90.5 mm
- net +3.3V: track 149.8 -> 150.7 mm
- net GND: track 0.00 -> 0.81 mm, vias 4 -> 2

Commit message: Changes to ulogger pcb
Parts:
- added BT1: Battery_Cell, Battery:BatteryHolder_Keystone_500, B.Cu at (108.6, 53.1)
- added Q2: 2N7002, Package_TO_SOT_SMD:SOT-23, F.Cu at (122.0, 79.3)
- added R3: 100k, Resistor_SMD:R_0805_2012Metric_Pad1.20x1.40mm_HandSolder, F.Cu at (121.1, 83.2)
- R1: value 100k -> 10k
- moved R2 6.43 mm to (126.9, 75.8)
- moved R_pullup_shtdwn1 6.01 mm to (131.2, 79.7), turned to 90 degrees
- moved P_MOSFET1 4.47 mm to (126.2, 71.7)
- moved R1 4.35 mm to (121.5, 75.9)
- moved C1 3.31 mm to (131.0, 72.9), turned to -90 degrees
- moved R_pullup_int1 3.07 mm to (126.7, 83.2)
- moved RpullupCS1 2.37 mm to (121.1, 96.2)
- moved C2 2.06 mm to (110.5, 82.9)
- moved PWRIN1 1.89 mm to (123.4, 49.4)
- moved U2 1.65 mm to (126.9, 79.7)
- moved C5 1.44 mm to (124.4, 62.5)
- moved SW2 1.24 mm to (130.9, 91.1)
- moved R_BYPASS1 1.12 mm to (126.8, 66.5), turned to 90 degrees
- moved Q1 1.04 mm to (129.6, 57.6)
- moved R8 0.78 mm to (126.3, 57.8)
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Connections:
- A1 pad 20: unconnected-(A1-GPIO15-Pad20) -> Net-(A1-GPIO15)
- A1 pad 27: Net-(A1-GPIO21) -> unconnected-(A1-GPIO21-Pad27)
- A1 pad 29: unconnected-(A1-GPIO22-Pad29) -> Net-(A1-GPIO22)
- J5 pad 2: unconnected-(J5-Pin_2-Pad2) -> Net-(A1-GPIO15)
- R1 pad 1: Net-(A1-GPIO21) -> Net-(A1-GPIO22)
- R1 pad 2: /SHTDWN_CTRL -> Net-(Q2-G)
- U1 pad 6: /BATT -> Net-(BT1-+)
Routing:
- net Net-(A1-GPIO15): track 0.00 -> 59.1 mm, vias 0 -> 2
- net /BATT: track 90.5 -> 32.6 mm
- net Net-(BT1-+): track 0.00 -> 16.7 mm, vias 0 -> 1
- net Net-(P_MOSFET1-G): track 9.76 -> 2.17 mm
- net /I2C0_SCL: track 96.9 -> 101.4 mm, vias 3 -> 2
- net Net-(A1-GPIO22): track 0.00 -> 3.42 mm
- net Net-(A1-GPIO21): track 3.27 -> 0.00 mm
- net Net-(Q2-G): track 0.00 -> 3.02 mm
- net Net-(Q2-S): track 0.00 -> 2.01 mm
- net /RTC_INT: track 83.2 -> 85.0 mm
- net +3.3V: track 150.7 -> 149.0 mm
- net /Data_Onewire: track 86.8 -> 88.3 mm
- net /I2C1_SDA: track 19.6 -> 18.3 mm
- net /CS: track 13.9 -> 15.2 mm, vias 0 -> 1
- net Net-(U2-1Y): track 3.95 -> 5.12 mm
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Other:
- board size 55 x 67 mm -> 60 x 67 mm
- board text added: "+"
- board text added: "-"
- board text added: "15"
- board text added: "1W"
- board text added: "3.3"
- board text added: "CL"
- board text added: "Cocoa-For-Flux µlogger"
- board text added: "DA"
- board text added: "G"
- board text added: "I2C 0"
- board text added: "I2C 1"
- board text added: "RX"
- board text added: "TX"

Commit message: Changes to small pcb
Parts:
- removed R_BYPASS1: 0 Ohm, Resistor_SMD:R_0805_2012Metric_Pad1.20x1.40mm_HandSolder
- added C3: 100 µF, Capacitor_THT:CP_Radial_D7.5mm_P2.50mm, F.Cu at (122.4, 59.8)
- C1, C4: footprint Capacitor_SMD:C_1812_4532Metric_Pad1.57x3.40mm_HandSolder -> Capacitor_SMD:C_1206_3216Metric_Pad1.33x1.80mm_HandSolder
- C5: value 100uF -> 10 µF
- moved C5 13.0 mm to (132.5, 72.6), turned to 0 degrees
- moved R3 9.61 mm to (124.3, 74.2), turned to 90 degrees
- moved PWRIN1 6.34 mm to (128.9, 46.3), turned to 180 degrees
- moved R8 4.28 mm to (124.9, 53.7), turned to 180 degrees
- moved C1 3.84 mm to (131.9, 76.7), turned to 0 degrees
- moved F1 3.74 mm to (130.3, 63.6)
- moved R_pullup_shtdwn1 3.73 mm to (130.5, 83.3), turned to 180 degrees
- moved Q1 2.77 mm to (129.1, 54.9)
- moved P_MOSFET1 2.06 mm to (125.9, 69.7)
- moved R2 1.58 mm to (127.0, 74.2)
- moved R_pullup_int1 1.20 mm to (125.5, 83.2)
- moved D1 1.15 mm to (121.3, 68.5)
- moved R1 0.86 mm to (121.2, 75.1)
- moved Q2 0.53 mm to (122.2, 78.8)
Connections:
- C5 pad 1: Net-(A1-VSYS) -> /BATT
- Q2 pad 2: Net-(Q2-S) -> GND
- R3 pad 1: Net-(Q2-S) -> Net-(Q2-G)
Routing:
- net +3.3V: track 149.0 -> 184.1 mm
- net /BATT: track 32.6 -> 43.4 mm, vias 2 -> 1
- net Net-(A1-VSYS): track 25.6 -> 19.3 mm
- net /I2C0_SCL: track 101.4 -> 104.2 mm
- net Net-(Q2-G): track 3.02 -> 5.23 mm
- net /I2C1_SCL: track 25.6 -> 23.6 mm
- net Net-(Q2-S): track 2.01 -> 0.00 mm
- net Net-(PWRIN1-Pin_2): track 8.47 -> 9.82 mm
- net /RTC_INT: track 85.0 -> 83.7 mm
- net Net-(A1-GPIO22): track 3.42 -> 2.25 mm
- net Net-(U2-1Y): track 5.12 -> 6.24 mm
- net Net-(Q1-S): track 3.74 -> 2.84 mm
- net /SHTDWN_CTRL: track 7.96 -> 7.07 mm
- net Net-(P_MOSFET1-G): track 2.17 -> 2.86 mm
- net Net-(Q1-G): track 2.45 -> 3.06 mm
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Other:
- board size 60 x 67 mm -> 63 x 67 mm
- board text added: "100k"
- board text added: "100nF"
- board text added: "100µF"
- board text added: "10k"
- board text added: "10µF"
- board text added: "1M"
- board text added: "2N7002"
- board text added: "PTC"
- board text added: "Pullup 1-Wire"
- board text added: "Pullups I2C1"
- board text added: "SN74"
- board text added: "SS14"
- board text added: "Si2301"
- board text added: "Switch ON"
